File: CcSoM_ADC_Board/CcSoM_ADC_Board.kicad_pcb (KiCad board)
At the start: 4 copper layers, 160 x 100 mm, 158 parts, among them J1 SoM Connector, J12 USB_C_Receptacle_USB2.0_16P, J13 Conn_02x03_Odd_Even, J14 Conn_02x03_Odd_Even, J15 Conn_02x02_Counter_Clockwise, J16 Barrel_Jack, J18 USB_A, J19 USB_A, J3 Conn_02x8_Odd_Even, J4 Conn_Coaxial, J5 HR911130A1, J6 Conn_01x14, J7 Conn_01x08, J8 Conn_01x16_Socket, J9 Conn_01x08, SW3 SW_Push, U1 SN74LVC00APWE4, U10 USB3343, U11 RTL8211E-VB-CG, U12 LTC2242IUP-12-PBF, U14 SN74CB3T3306DCTR, U2 74AUP1G04, U3 93LC46B, U4 FT2232HL, U5 SN74CB3T3245PWR, U6 TPS73625DBV, U7 TPS3307-33DR, U8 TPS73633DBV, X1 12MHz, Y1 25MHz

Commit message: last before rotating adc
Parts:
- added U9: TXS0202YZPR, TXS0202YZPR:YZP8, F.Cu at (167.8, 104.5)
Connections:
- J18 pad 2: USB2_- -> /usb2/D_+
- J18 pad 3: USB2_+ -> /usb2/D_-
Routing:
- net USB2_+: track 92.4 -> 41.5 mm
- net USB2_-: track 92.5 -> 41.6 mm
- net /usb2/D_-: track 0.00 -> 45.9 mm
- net /usb2/D_+: track 0.00 -> 45.9 mm
- net +3V3: track 453.0 -> 469.0 mm, vias 28 -> 29
- net OVDD: track 535.7 -> 538.9 mm, vias 32 -> 33
- net D3_N: track 31.8 -> 33.0 mm
- net D3_P: track 32.3 -> 33.4 mm
- net OGND: track 117.3 -> 118.4 mm, vias 258 -> 260
Other:
- board text added: "A"
- board text added: "Rev. 0.1 I Özdemirkan"
