File: CcSoM_ADC_Board/FTDI.kicad_sch (KiCad schematic)
At the start: 38 parts, among them J12 USB_C_Receptacle_USB2.0_16P, U14 SN74CB3T3306DCTR, U3 93LC46B, U4 FT2232HL, U5 SN74CB3T3245PWR, X1 12MHz

Commit message: corrected schematic created pdf and bom file
Other:
- moved on the sheet: C10, C13, C14, C2, C4, C5, C7, TP1, TP5

Commit message: changed schottky, began to add digikey part numbers
Parts:
- D17: footprint Diode_SMD:D_0402_1005Metric_Pad0.77x0.64mm_HandSolder -> Diode_SMD:D_0805_2012Metric_Pad1.15x1.40mm_HandSolder; DigiKey_no (none) -> 478-7800-1-ND
- R16: DigiKey_no (none) -> RMCF0603FT1K00CT-ND
- U14: DigiKey_no (none) -> 296-15553-1-ND
- U4: DigiKey_no (none) -> 768-1024-1-ND
- U5: DigiKey_no (none) -> 296-18196-1-ND
- X1: DigiKey_no (none) -> 300-8197-1-ND; MPN (none) -> ABM3B-12.000MHZ-10-1-U-T
Changed lines of the file:
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@@
 			)
 		)
+		(property "DigiKey_no" "RMCF0603FT1K00CT-ND"
+			(at 138.43 85.09 90)
+			(effects
+				(font
+					(size 1.27 1.27)
+				)
+				(hide yes)
+			)
+		)
 		(pin "1"
 		)
@@
 			)
 		)
-		(property "Footprint" "Diode_SMD:D_0402_1005Metric_Pad0.77x0.64mm_HandSolder"
+		(property "Footprint" "Diode_SMD:D_0805_2012Metric_Pad1.15x1.40mm_HandSolder"
 			(at 50.8 48.26 0)
 			(effects
@@
 			)
 		)
-		(property "Datasheet" "~"
+		(property "Datasheet" "https://datasheets.kyocera-avx.com/schottky.pdf"
 			(at 50.8 48.26 0)
 			(effects
@@
 			)
 		)
+		(property "DigiKey_no" "478-7800-1-ND"
+			(at 50.8 48.26 90)
+			(effects
+				(font
+					(size 1.27 1.27)
+				)
+				(hide yes)
+			)
+		)
 		(pin "1"
 		)
@@
 			)
 		)
+		(property "DigiKey_no" "296-15553-1-ND"
+			(at 223.52 104.14 0)
+			(effects
+				(font
+					(size 1.27 1.27)
+				)
+				(hide yes)
+			)
+		)
 		(pin "5"
 		)
@@
 			)
 		)
+		(property "DigiKey_no" "300-8197-1-ND"
+			(at 111.76 146.05 0)
+			(effects
+				(font
+					(size 1.27 1.27)
+				)
+				(hide yes)
+			)
+		)
+		(property "MPN" "ABM3B-12.000MHZ-10-1-U-T "
+			(at 111.76 146.05 0)
+			(effects
+				(font
+					(size 1.27 1.27)
+				)
+				(hide yes)
+			)
+		)
 		(pin "4"
 		)
@@
 			)
 		)
+		(property "DigiKey_no" "296-18196-1-ND"
+			(at 252.73 41.91 0)
+			(effects
+				(font
+					(size 1.27 1.27)
+				)
+				(hide yes)
+			)
+		)
 		(pin "16"
 		)
@@
 			(at 181.61 95.25 0)
 			(effects
+				(font
+					(size 1.27 1.27)
+				)
+				(hide yes)
+			)
+		)
+		(property "DigiKey_no" "768-1024-1-ND"
+			(at 181.61 95.25 0)
+			(effects

Commit message: digikey no not complete
Parts:
- C10, C13, C14, C2, C3, C4, C43, C5, C7, C9: DigiKey_no (none) -> 311-1088-1-ND
- C11, C8: DigiKey_no (none) -> 311-1058-1-ND
- C12: DigiKey_no (none) -> 399-3481-1-ND
- C59, C6: DigiKey_no (none) -> 490-7203-1-ND
- FB1, FB2: DigiKey_no (none) -> 445-MMZ1608R601ATD25CT-ND
- J12: DigiKey_no (none) -> 2073-USB4110-GF-A-1-ND
- R10, R11: DigiKey_no (none) -> 541-5.10KHCT-ND
- R12, R13, R14: DigiKey_no (none) -> 541-10.0KHCT-ND
- R15: DigiKey_no (none) -> 541-2.00KHCT-ND
- R17, R18: DigiKey_no (none) -> 541-12.0KHCT-ND
- U3: DigiKey_no (none) -> 93LC46BT-I/STCT-ND
