File: CcSoM_ADC_Board/HeaderInterface.kicad_sch (KiCad schematic)
At the start: 1 part, among them J3 Conn_02x8_Odd_Even

Commit message: corrected schematic created pdf and bom file
Other:
- title: SoM Programmer & Tester -> SoM Programmer & ADC Board
Changed lines of the file:
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@@
 	(paper "A4")
 	(title_block
-		(title "SoM Programmer & Tester")
+		(title "SoM Programmer & ADC Board")
 		(date "2024-12-20")
 		(rev "0.1")

Commit message: digikey no not complete
Parts:
- J3: DigiKey_no (none) -> 10129381-916001BLF-ND
Changed lines of the file:
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@@
+			)
+		)
+		(property "DigiKey_no" "10129381-916001BLF-ND"
+			(at 40.64 58.42 0)
+			(effects
+				(font
+					(size 1.27 1.27)
+				)
+				(hide yes)
 			)
 		)
