File: CcSoM_ADC_Board/PowerSupply.kicad_sch (KiCad schematic)
At the start: 14 parts, among them SW3 SW_Push, U6 TPS73625DBV, U7 TPS3307-33DR, U8 TPS73633DBV

Commit message: corrected schematic created pdf and bom file
Other:
- title: SoM Programmer & Tester -> SoM Programmer & ADC
Changed lines of the file:
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@@
 	(paper "A4")
 	(title_block
-		(title "SoM Programmer & Tester")
+		(title "SoM Programmer & ADC")
 		(date "2024-12-20")
 		(rev "0.1")

Commit message: changed schottky, began to add digikey part numbers
Parts:
- SW3: DigiKey_no (none) -> EG5353CT-ND
- U6: DigiKey_no (none) -> 296-39487-1-ND
- U7: DigiKey_no (none) -> 296-3314-1-ND
- U8: footprint ccsom_Footprint_lib:SOIC-8_5.8x3.81mm -> Package_TO_SOT_SMD:SOT-23-5; DigiKey_no (none) -> 296-52817-1-ND
Changed lines of the file:
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@@
+			)
+		)
+		(property "DigiKey_no" "296-39487-1-ND"
+			(at 80.01 45.72 0)
+			(effects
+				(font
+					(size 1.27 1.27)
+				)
+				(hide yes)
 			)
 		)
@@
 			)
 		)
+		(property "DigiKey_no" "296-3314-1-ND "
+			(at 130.81 113.03 0)
+			(effects
+				(font
+					(size 1.27 1.27)
+				)
+				(hide yes)
+			)
+		)
 		(pin "5"
 		)
@@
 			)
 		)
-		(property "Footprint" "ccsom_Footprint_lib:SOIC-8_5.8x3.81mm"
+		(property "Footprint" "Package_TO_SOT_SMD:SOT-23-5"
 			(at 223.52 36.195 0)
 			(effects
@@
 		)
 		(property "Mouser Price/Stock" "https://www.mouser.co.uk/ProductDetail/Texas-Instruments/TPS3307-33DR?qs=g%2FrhRe7LVpT4WdTNIYlIAw%3D%3D"
+			(at 223.52 44.45 0)
+			(effects
+				(font
+					(size 1.27 1.27)
+				)
+				(hide yes)
+			)
+		)
+		(property "DigiKey_no" "296-52817-1-ND"
 			(at 223.52 44.45 0)
 			(effects
@@
 			(at 185.42 115.57 0)
 			(effects
+				(font
+					(size 1.27 1.27)
+				)
+				(hide yes)
+			)
+		)
+		(property "DigiKey_no" "EG5353CT-ND"
+			(at 185.42 115.57 0)
+			(effects

Commit message: digikey no not complete
Parts:
- C15, C17, C18, C19, C21: DigiKey_no (none) -> 311-1088-1-ND
- C16, C20: DigiKey_no (none) -> 399-C0603C103K5RACTUCT-ND
- R19: DigiKey_no (none) -> 541-47.0KHCT-ND
- R20: DigiKey_no (none) -> 541-470KHCT-ND
- R21: DigiKey_no (none) -> 541-270KHCT-ND
Changed lines of the file:
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@@
+			)
+		)
+		(property "DigiKey_no" "541-47.0KHCT-ND"
+			(at 173.99 110.49 90)
+			(effects
+				(font
+					(size 1.27 1.27)
+				)
+				(hide yes)
 			)
 		)
@@
 			)
 		)
+		(property "DigiKey_no" "399-C0603C103K5RACTUCT-ND"
+			(at 236.22 50.8 0)
+			(effects
+				(font
+					(size 1.27 1.27)
+				)
+				(hide yes)
+			)
+		)
 		(pin "1"
 		)
@@
 			)
 		)
+		(property "DigiKey_no" "311-1088-1-ND"
+			(at 248.92 50.8 0)
+			(effects
+				(font
+					(size 1.27 1.27)
+				)
+				(hide yes)
+			)
+		)
 		(pin "1"
 		)
@@
 			)
 		)
+		(property "DigiKey_no" "311-1088-1-ND"
+			(at 104.14 49.53 0)
+			(effects
+				(font
+					(size 1.27 1.27)
+				)
+				(hide yes)
+			)
+		)
 		(pin "1"
 		)
@@
 			)
 		)
+		(property "DigiKey_no" "311-1088-1-ND"
+			(at 204.47 50.8 0)
+			(effects
+				(font
+					(size 1.27 1.27)
+				)
+				(hide yes)
+			)
+		)
 		(pin "1"
 		)
@@
 			)
 		)
+		(property "DigiKey_no" "399-C0603C103K5RACTUCT-ND"
+			(at 91.44 49.53 0)
+			(effects
+				(font
+					(size 1.27 1.27)
+				)
+				(hide yes)
+			)
+		)
 		(pin "1"
 		)
@@
 			)
 		)
+		(property "DigiKey_no" "541-470KHCT-ND"
+			(at 115.57 123.19 90)
+			(effects
+				(font
+					(size 1.27 1.27)
+				)
+				(hide yes)
+			)
+		)
 		(pin "2"
 		)
@@
 			)
 		)
+		(property "DigiKey_no" "541-270KHCT-ND"
+			(at 115.57 113.03 90)
+			(effects
+				(font
+					(size 1.27 1.27)
+				)
+				(hide yes)
+			)
+		)
 		(pin "2"
 		)
@@
 			)
 		)
+		(property "DigiKey_no" "311-1088-1-ND"
+			(at 59.69 49.53 0)
+			(effects
+				(font
+					(size 1.27 1.27)
+				)
+				(hide yes)
+			)
+		)
 		(pin "1"
 		)
@@
 			(at 167.64 127 0)
 			(effects
+				(font
+					(size 1.27 1.27)
+				)
+				(hide yes)
+			)
+		)
+		(property "DigiKey_no" "311-1088-1-ND"
+			(at 167.64 127 0)
+			(effects
